Commit message: att_camera

File: Ros-rep/my_robot_description/urdf/camera.xacro (robot description, xacro)
@@ -1,50 +1,59 @@
 <?xml version="1.0"?>
 <robot xmlns:xacro="http://www.ros.org/wiki/xacro">
-    <xacro:property name="camera_length" value="0.1" />
+    <xacro:property name="camera_length" value="0.01" />
     <xacro:property name="camera_width" value="0.1" />
     <xacro:property name="camera_height" value="0.05" />
-   <link name="camera_link">
-    <visual>
-        <geometry>
-            <box size="${camera_length} ${camera_width} ${camera_height}" />
-        </geometry>
-    </visual>
-    <collision>
-        <geometry>
-            <box size="${camera_length} ${camera_width} ${camera_height}" />
-        </geometry>
-    </collision>
-    <xacro:box_inertia m="0.1" x="${camera_length}" y="${camera_width}" z="${camera_height}" o_xyz="0 0 0" o_rpy="0 0 0" />
-   </link>
-   <joint name="base_camera_joint" type="fixed">
-    <parent link="base_link" />
-    <child link="camera_link" />
-    <origin xyz="${base_length/2.0} 0 ${base_height/2.0}" rpy="0 0 0" />
-   </joint>
-   <gazebo reference="camera_link">
-    <sensor name="camera" type="camera">
-  <camera>
-        <horizontal_fov>1.3962634</horizontal_fov>
-        <image>
-            <width>648</width>
-            <height>480</height>
-            <format>R8G8B8</format>
-        </image>
-        <clip>
-            <near>0.1</near>
-            <far>15</far>
-        </clip>
-        <noise>
-            <type>gaussian</type>
-            <mean>0.0</mean>
-            <stddev>0.007</stddev>
-        </noise>
-        <optical_frame_id>camera_link_optical</optical_frame_id>
-    </camera>
-        <always_on>1</always_on>
-        <update_rate>28</update_rate>
-        <visualize>true</visualize>
-        <topic>camera/image_raw</topic>
-    </sensor>
-   </gazebo>
+    <link name="camera_link">
+        <visual>
+            <geometry>
+                <box size="${camera_length} ${camera_width} ${camera_height}" />
+            </geometry>
+            <material name="grey" />
+        </visual>
+        <collision>
+            <geometry>
+                <box size="${camera_length} ${camera_width} ${camera_height}" />
+            </geometry>
+        </collision>
+        <xacro:box_inertia m="0.1" x="${camera_length}" y="${camera_width}" z="${camera_height}"
+                           o_xyz="0 0 0" o_rpy="0 0 0" />
+    </link>
+    <joint name="base_camera_joint" type="fixed">
+        <parent link="base_link" />
+        <child link="camera_link" />
+        <origin xyz="${(base_length + camera_length) / 2.0} 0 ${base_height / 2.0}" rpy="0 0 0" />
+    </joint>
+    <link name="camera_link_optical" />
+    <joint name="camera_optical_joint" type="fixed">
+        <origin xyz="0 0 0" rpy="${-pi/2} 0 ${-pi/2}"/>
+        <parent link="camera_link"/>
+        <child link="camera_link_optical"/>
+    </joint>
+    <gazebo reference="camera_link">
+        <sensor name="camera" type="camera">
+            <camera>
+                <horizontal_fov>1.3962634</horizontal_fov>
+                <image>
+                    <width>640</width>
+                    <height>480</height>
+                    <format>R8G8B8</format>
+                </image>
+                <clip>
+                    <near>0.1</near>
+                    <far>15</far>
+                </clip>
+                <noise>
+                    <type>gaussian</type>
+                    <mean>0.0</mean>
+                    <stddev>0.007</stddev>
+                </noise>
+                <optical_frame_id>camera_link_optical</optical_frame_id>
+                <camera_info_topic>camera/camera_info</camera_info_topic>
+            </camera>
+            <always_on>1</always_on>
+            <update_rate>20</update_rate>
+            <visualize>true</visualize>
+            <topic>camera/image_raw</topic>
+        </sensor>
+    </gazebo>
 </robot>
