Commit message: my_robot_final
Co-authored-by: Copilot <copilot@github.com>

File: Ros-rep/my_robot_description/urdf/common_properties.xacro (robot description, xacro)
@@ -1,10 +1,10 @@
 <?xml version="1.0"?>
 <robot xmlns:xacro="http://www.ros.org/wiki/xacro">
-    <material name="blue">
-        <color rgba="0 0 0.5 1" />
-    </material>
-    <material name="grey">
-        <color rgba="0.5 0.5 0.5 1" />
-    </material>
+  <material name="orange">
+    <color rgba="1.0 0.5 0.0 1.0"/>
+  </material>
+  <material name="yellow">
+    <color rgba="1.0 1.0 0.0 1.0"/>
+  </material>
     <xacro:macro name="box_inertia" params="m x y z o_xyz o_rpy">
         <inertial>

File: Ros-rep/my_robot_description/urdf/my_robot.urdf.xacro (robot description, xacro)
@@ -5,3 +5,41 @@
     <xacro:include filename="mobile_base_gazebo.xacro" />
     <xacro:include filename="camera.xacro" />
+    <xacro:include filename="arm.xacro" />
+    <xacro:include filename="arm_gazebo.xacro" />
+    <joint name="base_to_arm" type="fixed">
+        <parent link="base_link" />
+        <child link="arm_base_link" />
+        <origin xyz="${arm_base_length/4.0} 0 ${arm_base_height/2}" rpy="0 0 0" />
+    </joint>
+    <gazebo reference="base_link">
+    <visual>
+      <material>
+        <ambient>0.0 0.0 1.0 1.0</ambient> <diffuse>0.0 0.0 1.0 1.0</diffuse>
+        <specular>0.1 0.1 0.1 1.0</specular>
+      </material>
+    </visual>
+  </gazebo>
+  <gazebo reference="right_wheel_link">
+    <visual>
+      <material>
+        <ambient>0.2 0.2 0.2 1.0</ambient> <diffuse>0.2 0.2 0.2 1.0</diffuse>
+      </material>
+    </visual>
+  </gazebo>
+  <gazebo reference="left_wheel_link">
+    <visual>
+      <material>
+        <ambient>0.2 0.2 0.2 1.0</ambient>
+        <diffuse>0.2 0.2 0.2 1.0</diffuse>
+      </material>
+    </visual>
+  </gazebo>
+  <gazebo reference="caster_wheel_link">
+    <visual>
+      <material>
+        <ambient>0.2 0.2 0.2 1.0</ambient>
+        <diffuse>0.2 0.2 0.2 1.0</diffuse>
+      </material>
+    </visual>
+  </gazebo>
 </robot>
